File: PCB/attiny-e-ink/attiny-e-ink.kicad_pcb (KiCad board)
At the start: 2 copper layers, 52 x 32.1 mm, 31 parts, among them J1 e-ink-display, J2 Micro_SD_Card_Det_Hirose_DM3AT, J3 Battery, J4 USB4085-GF-A, Q1 DMG2301L, Q2 DMG2301L, Q3 DMG2301L, U1 ATtiny3226-S, U2 TPS7A0233PDBVR, U3 MCP73832

Commit message: check point
Parts:
- J3: footprint Connector:Alex_2pin_35thou -> molex-90-1.25:CONN02_530480210_MOL
- moved J3 0.59 mm to (160.0, 138.7), turned to 90 degrees
- moved J1 0.36 mm to (115.0, 118.1)
- moved S1 0.33 mm to (141.2, 111.9)
Connections:
- J3 pad 1: GND -> V_Bat
- J3 pad 2: V_Bat -> GND
Routing:
- net Net-(D1-A): track 24.4 -> 29.5 mm
- net V_Bat: track 34.9 -> 37.4 mm
- net GND: vias 37 -> 38
Other:
- board text removed: "+"
- board text removed: "-"
