File: PCB/attiny-e-ink/attiny-e-ink.kicad_sch (KiCad schematic)
At the start: 31 parts, among them J1 e-ink-display, J2 Micro_SD_Card_Det_Hirose_DM3AT, J3 Battery, J4 USB4085-GF-A, Q1 DMG2301L, Q2 DMG2301L, Q3 DMG2301L, U1 ATtiny3226-S, U2 TPS7A0233PDBVR, U3 MCP73832

Commit message: check point
Parts:
- J3: footprint Connector:Alex_2pin_35thou -> molex-90-1.25:CONN02_530480210_MOL
Connections:
- net GND: now also J3.2 (Pin_1); no longer J3.1 (Pin_1)
- net V_Bat: now also J3.1 (Pin_2); no longer J3.2 (Pin_2)
Changed lines of the file:
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@@
 			)
 		)
-		(property "Footprint" "Connector:Alex_2pin_35thou"
+		(property "Footprint" "molex-90-1.25:CONN02_530480210_MOL"
 			(at 194.31 69.85 0)
 			(hide yes)
